File: PowerBoard.kicad_sch (KiCad schematic)
At the start: 10 parts

Commit message: add additional AAM resistor and increment board version. Instructions for 3.3V output rather than 5V if desired.
Parts:
- added R4: 53.6K, Resistor_SMD:R_0603_1608Metric, symbol Device:R_Small_US
- Regulator5V1: footprint MPM3610AGQV-P:MPM3620AGQV-P -> CONV_MPM3620AGQV-P
- renumbered R2 to R1, R3 to R2, R1 to R3
Connections:
- net GND: now also R4.2
- net at Regulator5V1.18 (AAM): now also R4.1
- no-connect marks 3 -> 2
Changed lines of the file:
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@@
   (no_connect (at 187.96 80.01))
   (no_connect (at 218.44 64.77))
-  (no_connect (at 187.96 87.63))
   (wire (pts (xy 107.95 57.15) (xy 107.95 67.31))
     (stroke (width 0) (type default) (color 0 0 0 0))
@@
     (stroke (width 0) (type default) (color 0 0 0 0))
   )
+  (wire (pts (xy 187.96 87.63) (xy 184.15 87.63))
+    (stroke (width 0) (type default) (color 0 0 0 0))
+  )
   (wire (pts (xy 250.19 71.12) (xy 257.81 71.12))
     (stroke (width 0) (type default) (color 0 0 0 0))
@@
   )
   (wire (pts (xy 124.46 82.55) (xy 124.46 83.82))
+    (stroke (width 0) (type default) (color 0 0 0 0))
+  )
+  (wire (pts (xy 184.15 87.63) (xy 184.15 90.17))
     (stroke (width 0) (type default) (color 0 0 0 0))
   )
@@
   (symbol (lib_id "Device:R_Small_US") (at 232.41 83.82 0) (unit 1)
     (in_bom yes) (on_board yes) (fields_autoplaced)
-    (property "Reference" "R3" (id 0) (at 234.95 82.5499 0)
+    (property "Reference" "R2" (id 0) (at 234.95 82.5499 0)
       (effects (font (size 1.27 1.27)) (justify left))
     )
@@
     (pin "1")
   )
+  (symbol (lib_id "Device:R_Small_US") (at 184.15 92.71 0) (unit 1)
+    (in_bom yes) (on_board yes) (fields_autoplaced)
+    (property "Reference" "R4" (id 0) (at 186.69 91.4399 0)
+      (effects (font (size 1.27 1.27)) (justify left))
+    )
+    (property "Value" "53.6K" (id 1) (at 186.69 93.9799 0)
+      (effects (font (size 1.27 1.27)) (justify left))
+    )
+    (property "Footprint" "Resistor_SMD:R_0603_1608Metric" (id 2) (at 184.15 92.71 0)
+      (effects (font (size 1.27 1.27)) hide)
+    )
+    (property "Datasheet" "~" (id 3) (at 184.15 92.71 0)
+      (effects (font (size 1.27 1.27)) hide)
+    )
+    (pin "1")
+    (pin "2")
+  )
   (symbol (lib_id "power:GND") (at 55.88 72.39 90) (unit 1)
     (in_bom yes) (on_board yes) (fields_autoplaced)
@@
   (symbol (lib_id "Device:R_Small_US") (at 182.88 72.39 0) (unit 1)
     (in_bom yes) (on_board yes) (fields_autoplaced)
-    (property "Reference" "R1" (id 0) (at 185.42 71.1199 0)
+    (property "Reference" "R3" (id 0) (at 185.42 71.1199 0)
       (effects (font (size 1.27 1.27)) (justify left))
     )
@@
     (pin "2")
   )
-  (symbol (lib_name "MPM3610AGQV-P_1") (lib_id "MPM3610AGQV-P:MPM3610AGQV-P") (at 203.2 77.47 0) (unit 1)
+  (symbol (lib_id "MPM3610AGQV-P:MPM3610AGQV-P") (at 203.2 77.47 0) (unit 1)
     (in_bom yes) (on_board yes) (fields_autoplaced)
     (property "Reference" "Regulator5V1" (id 0) (at 203.2 57.15 0))
     (property "Value" "MPM3610AGQV-P" (id 1) (at 203.2 59.69 0))
-    (property "Footprint" "MPM3610AGQV-P:MPM3620AGQV-P" (id 2) (at 203.2 77.47 0)
+    (property "Footprint" "CONV_MPM3620AGQV-P" (id 2) (at 203.2 77.47 0)
       (effects (font (size 1.27 1.27)) (justify left bottom) hide)
     )
@@
     (pin "9")
   )
+  (symbol (lib_id "power:GND") (at 184.15 95.25 0) (unit 1)
+    (in_bom yes) (on_board yes) (fields_autoplaced)
+    (property "Reference" "#PWR0111" (id 0) (at 184.15 101.6 0)
+      (effects (font (size 1.27 1.27)) hide)
+    )
+    (property "Value" "GND" (id 1) (at 184.15 100.33 0))
+    (property "Footprint" "" (id 2) (at 184.15 95.25 0)
+      (effects (font (size 1.27 1.27)) hide)
+    )
+    (property "Datasheet" "" (id 3) (at 184.15 95.25 0)
+      (effects (font (size 1.27 1.27)) hide)
+    )
+    (pin "1")
+  )
   (symbol (lib_id "Device:R_Small_US") (at 232.41 73.66 0) (unit 1)
     (in_bom yes) (on_board yes) (fields_autoplaced)
-    (property "Reference" "R2" (id 0) (at 234.95 72.3899 0)
+    (property "Reference" "R1" (id 0) (at 234.95 72.3899 0)
       (effects (font (size 1.27 1.27)) (justify left))
     )
@@
       (reference "#PWR0110") (unit 1) (value "GND") (footprint "")
     )
+    (path "/e3a64cd0-0632-4b85-9a87-2a52308e6049"
+      (reference "#PWR0111") (unit 1) (value "GND") (footprint "")
+    )
     (path "/8e9d8fc8-7b5a-43f4-8fd7-f0b3c3cdc133"
       (reference "C1") (unit 1) (value "10uF") (footprint "")
@@
       (reference "PB1") (unit 1) (value "PowerBoard_Conn_01x05") (footprint "Connector_PinHeader_2.54mm:PinHeader_1x05_P2.54mm_Vertical")
     )
+    (path "/fb64ac3f-c3d1-4cef-8a6b-26a229dda872"
+      (reference "R1") (unit 1) (value "100K") (footprint "Resistor_SMD:R_0603_1608Metric")
+    )
+    (path "/600372f3-cdda-45ea-9e4e-4cb6464074bb"
+      (reference "R2") (unit 1) (value "19.1K") (footprint "Resistor_SMD:R_0603_1608Metric")
+    )
     (path "/abd58fa7-a9e2-4c2e-8c1b-3714a1fbec96"
-      (reference "R1") (unit 1) (value "100K") (footprint "Resistor_SMD:R_0603_1608Metric")
-    )
-    (path "/fb64ac3f-c3d1-4cef-8a6b-26a229dda872"
-      (reference "R2") (unit 1) (value "100K") (footprint "Resistor_SMD:R_0603_1608Metric")
-    )
-    (path "/600372f3-cdda-45ea-9e4e-4cb6464074bb"
-      (reference "R3") (unit 1) (value "19.1K") (footprint "Resistor_SMD:R_0603_1608Metric")
+      (reference "R3") (unit 1) (value "100K") (footprint "Resistor_SMD:R_0603_1608Metric")
+    )
+    (path "/95bbd89f-1fd7-4007-812c-242b3ddddb8d"
+      (reference "R4") (unit 1) (value "53.6K") (footprint "Resistor_SMD:R_0603_1608Metric")
     )
     (path "/46e4de66-b5e6-4fb5-9115-917ae09711e5"
@@
     )
     (path "/cb513a45-78a5-4b5b-9513-cde5c9d71318"
-      (reference "Regulator5V1") (unit 1) (value "MPM3610AGQV-P") (footprint "MPM3610AGQV-P:MPM3620AGQV-P")
-    )
-  )
+      (reference "Regulator5V1") (unit 1) (value "MPM3610AGQV-P") (footprint "CONV_MPM3620AGQV-P")
+    )
+  )

Commit message: version 1.2.
Parts:
- removed D1: D_Schottky, Diode_SMD:D_0603_1608Metric, symbol Device:D_Schottky
- added A0: A0, Jumper:SolderJumper-2_P1.3mm_Open_Pad1.0x1.5mm, symbol Jumper:SolderJumper_2_Open
- added A1: A1, Jumper:SolderJumper-2_P1.3mm_Open_Pad1.0x1.5mm, symbol Jumper:SolderJumper_2_Open
- added R5, R6: 10K, symbol Device:R_Small_US
Connections:
- net +5V: now also A0.2 (B), A1.2 (B)
- net GND: now also R5.2, R6.2; no longer CURRENT_MAIN1.1 (A1), CURRENT_MAIN1.2 (A0)
- net at CURRENT_MAIN1.8 (IN+), R_SHUNT1.1: now also PB1.1 (VCC)
- new net: A1.1 (A), CURRENT_MAIN1.1 (A1), R5.1
- new net: A0.1 (A), CURRENT_MAIN1.2 (A0), R6.1
Other:
- note added: "A1/A0 tied to ground equal I2C address = 0x40 Use the jumper to select different I2C addresses"
- note removed: "A1/A0 tied to ground equal I2C address = 0x40"

Commit message: update to 1.3.
Parts:
- C1, C2: footprint (none) -> Capacitor_SMD:C_0603_1608Metric_Pad1.08x0.95mm_HandSolder
- R5, R6: footprint (none) -> Resistor_SMD:R_0603_1608Metric
Changed lines of the file:
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@@
       (effects (font (size 1.27 1.27)) (justify left))
     )
-    (property "Footprint" "" (id 2) (at 250.19 80.01 0)
+    (property "Footprint" "Capacitor_SMD:C_0603_1608Metric_Pad1.08x0.95mm_HandSolder" (id 2) (at 250.19 80.01 0)
       (effects (font (size 1.27 1.27)) hide)
     )
@@
       (effects (font (size 1.27 1.27)) (justify left))
     )
-    (property "Footprint" "" (id 2) (at 132.08 88.9 0)
+    (property "Footprint" "Resistor_SMD:R_0603_1608Metric" (id 2) (at 132.08 88.9 0)
       (effects (font (size 1.27 1.27)) hide)
     )
@@
       (effects (font (size 1.27 1.27)) (justify left))
     )
-    (property "Footprint" "" (id 2) (at 123.19 88.9 0)
+    (property "Footprint" "Resistor_SMD:R_0603_1608Metric" (id 2) (at 123.19 88.9 0)
       (effects (font (size 1.27 1.27)) hide)
     )
@@
       (effects (font (size 1.27 1.27)) (justify left))
     )
-    (property "Footprint" "" (id 2) (at 168.91 74.93 0)
+    (property "Footprint" "Capacitor_SMD:C_0603_1608Metric_Pad1.08x0.95mm_HandSolder" (id 2) (at 168.91 74.93 0)
       (effects (font (size 1.27 1.27)) hide)
     )
@@
     )
     (path "/8e9d8fc8-7b5a-43f4-8fd7-f0b3c3cdc133"
-      (reference "C1") (unit 1) (value "10uF") (footprint "")
+      (reference "C1") (unit 1) (value "10uF") (footprint "Capacitor_SMD:C_0603_1608Metric_Pad1.08x0.95mm_HandSolder")
     )
     (path "/02d81d42-15f4-4cda-b8eb-2c773fa1cca1"
-      (reference "C2") (unit 1) (value "22uF") (footprint "")
+      (reference "C2") (unit 1) (value "22uF") (footprint "Capacitor_SMD:C_0603_1608Metric_Pad1.08x0.95mm_HandSolder")
     )
     (path "/02dbc2e1-68de-439f-bfec-4d6d66d36a0f"
@@
     )
     (path "/8b72dcf0-166b-4eaf-90d8-721d7ec31645"
-      (reference "R5") (unit 1) (value "10K") (footprint "")
+      (reference "R5") (unit 1) (value "10K") (footprint "Resistor_SMD:R_0603_1608Metric")
     )
     (path "/4cde5e32-d245-434b-a5dc-3465a9af0c92"
-      (reference "R6") (unit 1) (value "10K") (footprint "")
+      (reference "R6") (unit 1) (value "10K") (footprint "Resistor_SMD:R_0603_1608Metric")
     )
     (path "/46e4de66-b5e6-4fb5-9115-917ae09711e5"
